Commit message: fix URDF

File: harvest_studio_description/urdf/harvest_studio.urdf.xacro (robot description, xacro)
@@ -89,18 +89,17 @@
   </link>
   <joint
-    name="azure_camera_joint"
-    type="fixed">
-    <origin
-      xyz="0.00385 0.465 0.98"
-      rpy="0 0 -3.1416" />
-    <parent
-      link="stand_base" />
-    <child
-      link="azure_camera_link" />
-    <axis
-      xyz="1 0 0" />
+   name="azure_camera_joint"
+   type="revolute">
+    <origin
+     xyz="0.00385 0.465 0.98"
+     rpy="0 0 -3.1416" />
+    <parent
+     link="stand_base" />
+    <child
+     link="azure_camera_link" />
+    <axis xyz="1 0 0" />
     <limit
-      lower="-0.5"
-      upper="0.5"
+     lower="-0.5"
+     upper="0.5"
       effort="0"
       velocity="0" />
@@ -148,5 +147,5 @@
   <joint
     name="right_arm_joint"
-    type="fixed">
+    type="revolute">
     <origin
       xyz="-0.30665 -0.4925 -0.155"
@@ -157,5 +156,5 @@
       link="right_arm_link" />
     <axis
-      xyz="0 1 0" />
+      xyz="0 0 1" />
     <limit
       lower="-1"
@@ -206,5 +205,5 @@
   <joint
     name="left_arm_joint"
-    type="fixed">
+    type="revolute">
     <origin
       xyz="0.30835 -0.505 -0.155"
@@ -215,5 +214,5 @@
       link="left_arm_link" />
     <axis
-      xyz="0 1 0" />
+      xyz="0 0 1" />
     <limit
       lower="-1"

Commit message: add ros2_xarm

File: harvest_studio_description/urdf/harvest_studio.urdf.xacro (robot description, xacro)
@@ -1,329 +1,16 @@
-<?xml version="1.0" encoding="utf-8"?>
-<robot
-  name="harvest-studio" xmlns:xacro="http://ros.org/wiki/xacro">
-  <link name="dummy">
-  </link>
-  <link
-    name="stand_base">
-    <inertial>
-      <origin
-        xyz="-0.00244095696499763 0.0834846502705878 0.0120971081555862"
-        rpy="0 0 0" />
-      <mass
-        value="17.4192822915786" />
-      <inertia
-        ixx="0.365207090762505"
-        ixy="1.51826662793011E-05"
-        ixz="-4.58049242566518E-08"
-        iyy="0.347003054917912"
-        iyz="-5.19603726593645E-07"
-        izz="0.177730015853551" />
-    </inertial>
-    <visual>
-      <origin
-        xyz="0 0 0"
-        rpy="0 0 0" />
-      <geometry>
-        <mesh
-          filename="file:///$(find harvest_studio_description)/stand_base.STL" />
-      </geometry>
-      <material
-        name="">
-        <color
-          rgba="0.752941176470588 0.752941176470588 0.752941176470588 1" />
-      </material>
-    </visual>
-    <collision>
-      <origin
-        xyz="0 0 0"
-        rpy="0 0 0" />
-      <geometry>
-        <mesh
-          filename="file:///$(find harvest_studio_description)/stand_base.STL" />
-      </geometry>
-    </collision>
-  </link>
-    <joint name="dummy_joint" type="fixed">
-    <parent link="dummy"/>
-    <child link="stand_base"/>
-  </joint>
-  <link
-    name="azure_camera_link">
-    <inertial>
-      <origin
-        xyz="-2.657383322537E-06 0.00348132910528381 0.0446566695341433"
-        rpy="0 0 0" />
-      <mass
-        value="2.78889236681522" />
-      <inertia
-        ixx="0.00412183232658945"
-        ixy="4.09236432683366E-07"
-        ixz="-3.17078316364308E-08"
-        iyy="0.00242404662476713"
-        iyz="0.000234310769319999"
-        izz="0.00609587810828995" />
-    </inertial>
-    <visual>
-      <origin
-        xyz="0 0 0"
-        rpy="0 0 0" />
-      <geometry>
-        <mesh
-          filename="file:///$(find harvest_studio_description)/azure_camera_link.STL" />
-      </geometry>
-      <material
-        name="">
-        <color
-          rgba="0.792156862745098 0.819607843137255 0.933333333333333 1" />
-      </material>
-    </visual>
-    <collision>
-      <origin
-        xyz="0 0 0"
-        rpy="0 0 0" />
-      <geometry>
-        <mesh
-          filename="file:///$(find harvest_studio_description)/azure_camera_link.STL" />
-      </geometry>
-    </collision>
-  </link>
-  <joint
-   name="azure_camera_joint"
-   type="revolute">
-    <origin
-     xyz="0.00385 0.465 0.98"
-     rpy="0 0 -3.1416" />
-    <parent
-     link="stand_base" />
-    <child
-     link="azure_camera_link" />
-    <axis xyz="1 0 0" />
-    <limit
-     lower="-0.5"
-     upper="0.5"
-      effort="0"
-      velocity="0" />
-  </joint>
-  <link
-    name="right_arm_link">
-    <inertial>
-      <origin
-        xyz="-0.0921692043278863 0.101109637912098 -0.00094798511080818"
-        rpy="0 0 0" />
-      <mass
-        value="0.879635804902705" />
-      <inertia
-        ixx="0.00101359963830436"
-        ixy="0.000345626145803582"
-        ixz="1.59140398416402E-07"
-        iyy="0.00110135479443889"
-        iyz="7.17570599023293E-08"
-        izz="0.000932982342715155" />
-    </inertial>
-    <visual>
-      <origin
-        xyz="0 0 0"
-        rpy="0 0 0" />
-      <geometry>
-        <mesh
-          filename="file:///$(find harvest_studio_description)/right_arm_link.STL" />
-      </geometry>
-      <material
-        name="">
-        <color
-          rgba="0.792156862745098 0.819607843137255 0.933333333333333 1" />
-      </material>
-    </visual>
-    <collision>
-      <origin
-        xyz="0 0 0"
-        rpy="0 0 0" />
-      <geometry>
-        <mesh
-          filename="file:///$(find harvest_studio_description)/right_arm_link.STL" />
-      </geometry>
-    </collision>
-  </link>
-  <joint
-    name="right_arm_joint"
-    type="revolute">
-    <origin
-      xyz="-0.30665 -0.4925 -0.155"
-      rpy="3.1416 0 0.90153" />
-    <parent
-      link="stand_base" />
-    <child
-      link="right_arm_link" />
-    <axis
-      xyz="0 0 1" />
-    <limit
-      lower="-1"
-      upper="1"
-      effort="0"
-      velocity="0" />
-  </joint>
-  <link
-    name="left_arm_link">
-    <inertial>
-      <origin
-        xyz="-0.13125187743035 0.0386239273471152 0.000950962918044584"
-        rpy="0 0 0" />
-      <mass
-        value="0.879657265086363" />
-      <inertia
-        ixx="0.00073064298535606"
-        ixy="0.000120666064530641"
-        ixz="-9.10646468836211E-08"
-        iyy="0.00138432044490653"
-        iyz="-1.38587279405028E-07"
-        izz="0.000932986858091463" />
-    </inertial>
-    <visual>
-      <origin
-        xyz="0 0 0"
-        rpy="0 0 0" />
-      <geometry>
-        <mesh
-          filename="file:///$(find harvest_studio_description)/left_arm_link.STL" />
-      </geometry>
-      <material
-        name="">
-        <color
-          rgba="0.792156862745098 0.819607843137255 0.933333333333333 1" />
-      </material>
-    </visual>
-    <collision>
-      <origin
-        xyz="0 0 0"
-        rpy="0 0 0" />
-      <geometry>
-        <mesh
-          filename="file:///$(find harvest_studio_description)/left_arm_link.STL" />
-      </geometry>
-    </collision>
-  </link>
-  <joint
-    name="left_arm_joint"
-    type="revolute">
-    <origin
-      xyz="0.30835 -0.505 -0.155"
-      rpy="0 0 1.6946" />
-    <parent
-      link="stand_base" />
-    <child
-      link="left_arm_link" />
-    <axis
-      xyz="0 0 1" />
-    <limit
-      lower="-1"
-      upper="1"
-      effort="0"
-      velocity="0" />
-  </joint>
-  <link
-    name="xArm_5_Lite">
-    <inertial>
-      <origin
-        xyz="-0.571524666474263 0.299537834362898 -0.192017553596648"
-        rpy="0 0 0" />
-      <mass
-        value="8.12684778121861" />
-      <inertia
-        ixx="0.0317436535196432"
-        ixy="8.74294723952674E-05"
-        ixz="-0.000698945548526394"
-        iyy="0.0145155514854216"
-        iyz="-0.00266520428215521"
-        izz="0.0333350986714747" />
-    </inertial>
-    <visual>
-      <origin
-        xyz="0 0 0"
-        rpy="0 0 0" />
-      <geometry>
-        <mesh
-          filename="file:///$(find harvest_studio_description)/xArm_5_Lite.STL" />
-      </geometry>
-      <material
-        name="">
-        <color
-          rgba="0.752941176470588 0.752941176470588 0.752941176470588 1" />
-      </material>
-    </visual>
-    <collision>
-      <origin
-        xyz="0 0 0"
-        rpy="0 0 0" />
-      <geometry>
-        <mesh
-          filename="file:///$(find harvest_studio_description)/xArm_5_Lite.STL" />
-      </geometry>
-    </collision>
-  </link>
-  <joint
-    name="xarm_joint"
-    type="fixed">
-    <origin
-      xyz="0.4659 0.34412 0.015649"
-      rpy="1.5708 0 1.0472" />
-    <parent
-      link="stand_base" />
-    <child
-      link="xArm_5_Lite" />
-    <axis
-      xyz="0 0 0" />
-  </joint>
-  <link
-    name="end_effector">
-    <inertial>
-      <origin
-        xyz="-9.11500058244363E-05 0.00639552591800449 -0.001811197649131"
-        rpy="0 0 0" />
-      <mass
-        value="0.49484420134997" />
-      <inertia
-        ixx="0.000184779666763685"
-        ixy="-6.20479155585265E-08"
-        ixz="-1.82180240805302E-06"
-        iyy="0.000219324560796222"
-        iyz="-1.12666169067249E-07"
-        izz="0.000188487226347135" />
-    </inertial>
-    <visual>
-      <origin
-        xyz="0 0 0"
-        rpy="0 0 0" />
-      <geometry>
-        <mesh
-          filename="file:///$(find harvest_studio_description)/end_effector.STL" />
-      </geometry>
-      <material
-        name="">
-        <color
-          rgba="0.752941176470588 0.752941176470588 0.752941176470588 1" />
-      </material>
-    </visual>
-    <collision>
-      <origin
-        xyz="0 0 0"
-        rpy="0 0 0" />
-      <geometry>
-        <mesh
-          filename="file:///$(find harvest_studio_description)/end_effector.STL" />
-      </geometry>
-    </collision>
-  </link>
-  <joint
-    name="end_effector_joint"
-    type="fixed">
-    <origin
-      xyz="-0.7103 0 -0.12789"
-      rpy="0 0 3.1416" />
-    <parent
-      link="xArm_5_Lite" />
-    <child
-      link="end_effector" />
-    <axis
-      xyz="0 0 0" />
-  </joint>
+<robot name="automato-robot" xmlns:xacro="thhp://ros.org/wiki/xacro">
+    <xacro:arg name="dof" default="5"/>
+    <xacro:include filename="$(find harvest_studio_description)/harvest_studio_robot.urdf.xacro"/>
+    <xacro:include filename="$(find xarm_description)/urdf/xarm_device.urdf.xacro"/>
+    <xacro:include filename="$(find harvest_studio_description)/harvest_studio_endeffector.urdf.xacro"/>
+    <joint name="arm_stand_joint" type="fixed">
+        <origin rpy="0 0 -1.57" xyz="0 0 0"/>
+        <parent link="stand_base"/>
+        <child link="world"/>
+    </joint>
+    <joint name="arm_eef_joint" type="fixed">
+        <origin rpy="1.57 0 0" xyz="0 0 0.097"/>
+        <parent link="link_eef"/>
+        <child link="end_effector"/>
+    </joint>
 </robot>

Commit message: update dynamixel control

File: harvest_studio_description/urdf/harvest_studio.urdf.xacro (robot description, xacro)
@@ -1,6 +1,6 @@
-<robot name="automato-robot" xmlns:xacro="thhp://ros.org/wiki/xacro">
+<robot name="" xmlns:xacro="thhp://ros.org/wiki/xacro">
     <xacro:arg name="dof" default="5"/>
+    <xacro:include filename="$(find xarm_description)/urdf/xarm_device.urdf.xacro"/>-->
     <xacro:include filename="$(find harvest_studio_description)/harvest_studio_robot.urdf.xacro"/>
-    <xacro:include filename="$(find xarm_description)/urdf/xarm_device.urdf.xacro"/>
     <xacro:include filename="$(find harvest_studio_description)/harvest_studio_endeffector.urdf.xacro"/>
     <joint name="arm_stand_joint" type="fixed">

File: harvest_studio_description/urdf/harvest_studio_robot.urdf.xacro (robot description, xacro)
@@ -1,5 +1,5 @@
 <?xml version="1.0" encoding="utf-8"?>
 <robot
-  name="harvest-studio" xmlns:xacro="http://ros.org/wiki/xacro">
+  name="harvest_studio" xmlns:xacro="http://ros.org/wiki/xacro">
   <link name="dummy">
   </link>

File: xarm_ros2/xarm_description/urdf/xarm_device_macro.xacro (robot description, xacro)
@@ -61,4 +61,5 @@
       />
     </xacro:if>
+    <!--<xacro:include filename="$(find harvest_studio_description)/harvest_studio.urdf.xacro"/>-->
   </xacro:macro>
 </robot>

File: xarm_ros2/xarm_moveit_config/srdf/_xarm5_macro.srdf.xacro (robot description, xacro)
@@ -33,9 +33,10 @@
       </xacro:if>
     </group>
-    <group name="harvest_studio">
+  <!--<group name="harvest_studio">
       <joint name="azure_camera_joint"/>
+      <joint name="arm_stand_joint"/>
       <joint name="right_arm_joint"/>
-      <joint name="left_arm_joint"/>
-    </group>
+      <joint name="left_arm_joint" />
+    </group>-->
     <!-- GROUP STATES, Purpose, Define a named state for a particular group, in terms of joint values. This is useful to define states like 'folded arms' -->
     <group_state name="home" group="${prefix}xarm5">
@@ -52,9 +53,4 @@
       <joint name="${prefix}joint4" value="-1.5708" />
       <joint name="${prefix}joint5" value="0" />
-    </group_state>
-    <group_state name="home" group="harvest_studio">
-      <joint name="azure_camera_joint" value="0"/>
-      <joint name="right_arm_joint" value="0"/>
-      <joint name="left_arm_joint" value="0"/>
     </group_state>
     <!-- gripper -->
@@ -151,4 +147,8 @@
     <disable_collisions link1="${prefix}link3" link2="${prefix}link5" reason="Never" />
     <disable_collisions link1="${prefix}link4" link2="${prefix}link5" reason="Adjacent" />
+    <!--<disable_collisions link1="stand_base" link2="${prefix}link1" reason="Adjacent" />
+    <disable_collisions link1="stand_base" link2="azure_camera_link" reason="Adjacent" />
+    <disable_collisions link1="stand_base" link2="right_arm_link" reason="Adjacent" />
+    <disable_collisions link1="stand_base" link2="left_arm_link" reason="Adjacent" /> -->
   </xacro:macro>
 </robot>

Commit message: なぜかxarmがros2で動いた

File: harvest_studio_description/urdf/harvest_studio.urdf.xacro (robot description, xacro)
@@ -1,7 +1,7 @@
 <robot name="" xmlns:xacro="thhp://ros.org/wiki/xacro">
     <xacro:arg name="dof" default="5"/>
-    <!--<xacro:include filename="$(find xarm_description)/urdf/xarm_device.urdf.xacro"/>-->
+    <xacro:include filename="$(find xarm_description)/urdf/xarm_device.urdf.xacro"/>
     <xacro:include filename="$(find harvest_studio_description)/harvest_studio_robot.urdf.xacro"/>
-    <xacro:include filename="$(find harvest_studio_description)/harvest_studio_endeffector.urdf.xacro"/>
+    <!--<xacro:include filename="$(find harvest_studio_description)/harvest_studio_endeffector.urdf.xacro"/>-->
     <joint name="arm_stand_joint" type="fixed">
         <origin rpy="0 0 -1.57" xyz="0 0 0"/>
@@ -9,8 +9,8 @@
         <child link="world"/>
     </joint>
-    <joint name="arm_eef_joint" type="fixed">
+    <!--<joint name="arm_eef_joint" type="fixed">
         <origin rpy="1.57 0 0" xyz="0 0 0.097"/>
         <parent link="link_eef"/>
         <child link="end_effector"/>
-    </joint>
+    </joint>-->
 </robot>

File: harvest_studio_description/urdf/harvest_studio_robot.urdf.xacro (robot description, xacro)
@@ -2,6 +2,4 @@
 <robot
   name="harvest_studio" xmlns:xacro="http://ros.org/wiki/xacro">
-  <link name="dummy">
-  </link>
   <link
     name="stand_base">
@@ -44,8 +42,4 @@
     </collision>
   </link>
-    <joint name="dummy_joint" type="fixed">
-    <parent link="dummy"/>
-    <child link="stand_base"/>
-  </joint>
   <link
     name="azure_camera_link">

Commit message: xarm was controlled by moveit api

File: harvest_studio_description/urdf/harvest_studio.urdf.xacro (robot description, xacro)
@@ -5,7 +5,7 @@
     <!--<xacro:include filename="$(find harvest_studio_description)/harvest_studio_endeffector.urdf.xacro"/>-->
     <joint name="arm_stand_joint" type="fixed">
-        <origin rpy="0 0 -1.57" xyz="0 0 0"/>
-        <parent link="stand_base"/>
-        <child link="world"/>
+        <origin rpy="0 0 1.57" xyz="0 0 0"/>
+        <parent link="world"/>
+        <child link="stand_base"/>
     </joint>
     <!--<joint name="arm_eef_joint" type="fixed">
